File: Cable.sch (KiCad schematic (older format))
At the start: 122 parts

Commit message: Add Cables
Parts:
- WIRE? (x4): KICABLE_HEADER:Cable-Length 6\" -> ?\"
Connections:
- net at WIRE?.1: now also J?.1 (Pin_1); no longer J?.4 (Pin_4) (x2)
- net at WIRE?.3: now also J?.2 (Pin_2); no longer J?.3 (Pin_3) (x2)
- net at WIRE?.5: now also J?.3 (Pin_3); no longer J?.2 (Pin_2) (x2)
- net at WIRE?.7: now also J?.4 (Pin_4); no longer J?.1 (Pin_1) (x2)
- no-connect marks 34 -> 35
Other:
- note added: "A+"
- note added: "A-"
- note added: "B+"
- note added: "B-"
- note added: "blu"
- note added: "grn"
- note added: "wht"
- note added: "ylw"
- moved on the sheet: J?
